File: EthernetTestBoard.kicad_pcb (KiCad board)
At the start: 2 copper layers, 51.4 x 71.7 mm, 43 parts, among them J1 USB_C_Receptacle, P1 RB1-125BAG1A, Q1 BC817-40_215, Q2 BC817-40_215, U1 ESP32-WROOM-E, U2 W5500, U3 CP2102N-Axx-xQFN24, U4 MIC5365-3.3YC5-TR, Y1 Crystal

Commit message: impedance matching match match
Parts:
- added R18: 100, Capacitor_SMD:C_0603_1608Metric_Pad1.08x0.95mm_HandSolder, F.Cu at (133.5, 77.3)
- added R19: 100, Capacitor_SMD:C_0603_1608Metric_Pad1.08x0.95mm_HandSolder, F.Cu at (138.1, 80.3)
- moved C9 2.77 mm to (124.0, 99.5)
Connections:
- C1 pad 2: GNDA -> GND
- C7 pad 1: VDDA -> +3V3
- C7 pad 2: GNDA -> GND
- C8 pad 2: GNDA -> GND
- C9 pad 2: GNDA -> GND
- R10 pad 1: VDDA -> +3V3
- R11 pad 1: VDDA -> +3V3
- R6 pad 1: GNDA -> GND
- U2 pad 1: /TD- -> Net-(U2-Pad1)
- U2 pad 11: VDDA -> +3V3
- U2 pad 14: GNDA -> GND
- U2 pad 15: VDDA -> +3V3
- U2 pad 16: GNDA -> GND
- U2 pad 17: VDDA -> +3V3
- U2 pad 19: GNDA -> GND
- U2 pad 2: /TD+ -> Net-(U2-Pad2)
- U2 pad 21: VDDA -> +3V3
- U2 pad 3: GNDA -> GND
- U2 pad 4: VDDA -> +3V3
- U2 pad 48: GNDA -> GND
- U2 pad 8: VDDA -> +3V3
- U2 pad 9: GNDA -> GND
Routing:
- net +3V3: track 161.9 -> 230.4 mm
- net GND: track 230.4 -> 293.5 mm, vias 11 -> 15
- net GNDA: track 60.3 -> 0.00 mm, vias 4 -> 0
- net VDDA: track 58.6 -> 0.00 mm
- net Net-(U2-Pad2): track 0.00 -> 8.40 mm
- net Net-(U2-Pad1): track 0.00 -> 8.33 mm
- net Net-(C9-Pad1): track 9.44 -> 12.2 mm
- net /TD-: track 31.3 -> 30.4 mm
- net Net-(R15-Pad2): track 39.3 -> 40.1 mm
- added copper zone on In1.Cu, net (none)
- added copper zone on In2.Cu, net (none)
Other:
- copper layers 2 -> 4

Commit message: lemme go home
Parts:
- removed U4: MIC5365-3.3YC5-TR, MIC5365-3:SOT65P210X110-5N
- added C13: 1uF, Capacitor_SMD:C_1812_4532Metric_Pad1.57x3.40mm_HandSolder, B.Cu at (97.0, 86.5)
- added C14: 0.1uF, Capacitor_SMD:C_1812_4532Metric_Pad1.57x3.40mm_HandSolder, B.Cu at (96.8, 75.9)
- added C15: 10nF, Capacitor_SMD:C_1812_4532Metric_Pad1.57x3.40mm_HandSolder, B.Cu at (103.1, 76.9)
- added R20: 10K, Resistor_SMD:R_0805_2012Metric_Pad1.20x1.40mm_HandSolder, B.Cu at (136.0, 76.2)
- added R21: 10K, Resistor_SMD:R_0805_2012Metric_Pad1.20x1.40mm_HandSolder, B.Cu at (139.3, 76.4)
- added R22: 10K, Resistor_SMD:R_0805_2012Metric_Pad1.20x1.40mm_HandSolder, B.Cu at (141.4, 84.3)
- added VR1: AP7366-33W5-7, AP7366-33W5-7:SOT95P285X140-5N, B.Cu at (96.1, 81.3)
- C10: value 7.14nF -> 0.1uF; footprint Capacitor_SMD:C_1206_3216Metric_Pad1.33x1.80mm_HandSolder -> Capacitor_SMD:C_0603_1608Metric_Pad1.08x0.95mm_HandSolder; moved to B.Cu
- C12, R18: moved to B.Cu
- R51, R52: value 5K -> 5.1K
- moved C10 39.6 mm to (140.7, 87.3), turned to 90 degrees
- moved R18 3.52 mm to (130.9, 74.9), turned to 0 degrees
- moved R19 1.05 mm to (137.7, 79.3)
- moved C12 0.35 mm to (103.4, 85.7)
- moved J1 0.28 mm to (118.6, 136.7)
Connections:
- C10 pad 1: +3V3 -> Net-(U3-Pad5)
- R5 pad 1: +3V3 -> /INTN
- U1 pad 14: unconnected-(U1-Pad14) -> /INTN
- U2 pad 43: Net-(U2-Pad43) -> /PMODE2
- U2 pad 44: Net-(U2-Pad43) -> /PMODE1
- U2 pad 45: Net-(U2-Pad43) -> /PMODE0
- U3 pad 5: GND -> Net-(U3-Pad5)
- U3 pad 6: GND -> Net-(U3-Pad5)
Routing:
- net Net-(C3-Pad1): track 57.6 -> 152.6 mm, vias 2 -> 4
- net GND: track 293.5 -> 220.9 mm, vias 15 -> 19
- net Net-(U3-Pad5): track 0.00 -> 52.9 mm, vias 0 -> 3
- net +3V3: track 230.4 -> 184.8 mm, vias 5 -> 11
- net /INTN: track 0.00 -> 31.5 mm, vias 0 -> 1
- net /EN: track 7.72 -> 38.7 mm, vias 0 -> 1
- net Net-(R9-Pad1): track 0.00 -> 24.1 mm, vias 0 -> 3
- net /PMODE0: track 0.00 -> 15.5 mm, vias 0 -> 4
- net /PMODE1: track 0.00 -> 13.2 mm, vias 0 -> 3
- net /PMODE2: track 0.00 -> 11.1 mm, vias 0 -> 3
- net Net-(R18-Pad1): track 8.40 -> 17.1 mm, vias 0 -> 1
- net /RD+: track 34.7 -> 38.4 mm, vias 0 -> 1
- net Net-(C12-Pad1): track 11.3 -> 15.0 mm, vias 1 -> 2
- net Net-(J1-PadA6): track 24.0 -> 27.2 mm
- net Net-(J1-PadA7): track 17.3 -> 20.4 mm
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- added copper zone on In2.Cu, net +3V3
- added copper zone on In1.Cu, net GND
- removed copper zone on In1.Cu, net (none)
- removed copper zone on In2.Cu, net (none)
