File: EthernetTestBoard.kicad_sch (KiCad schematic)
At the start: 42 parts, among them J1 USB_C_Receptacle, P1 RB1-125BAG1A, Q1 BC817-40_215, Q2 BC817-40_215, U1 ESP32-WROOM-E, U2 W5500, U3 CP2102N-Axx-xQFN24, U4 MIC5365-3.3YC5-TR, Y1 Crystal

Commit message: impedance matching match match
Parts:
- added R18, R19: 100, Capacitor_SMD:C_0603_1608Metric_Pad1.08x0.95mm_HandSolder, symbol Device:R
Connections:
- net GNDA is gone; now on net GND: C1.2, C7.2, C8.2, C9.2, R6.1, U2.14 (AGND), U2.16 (AGND), U2.19 (AGND), U2.3 (AGND), U2.48 (AGND), U2.9 (AGND)
- net VDDA is gone; now on net +3V3: C7.1, R10.1, R11.1, U2.11 (AVDD), U2.15 (AVDD), U2.17 (AVDD), U2.21 (AVDD), U2.4 (AVDD), U2.8 (AVDD)
- net TD+: now also R18.2; no longer U2.2 (TXP)
- net TD-: now also R19.2; no longer U2.1 (TXN)
- new net: R19.1, U2.1 (TXN)
- new net: R18.1, U2.2 (TXP)

Commit message: lemme go home
Parts:
- removed U4: MIC5365-3.3YC5-TR, MIC5365-3:SOT65P210X110-5N, symbol MIC5365-3.3YC5-TR:MIC5365-3.3YC5-TR
- added C13: 1uF, Capacitor_SMD:C_1812_4532Metric_Pad1.57x3.40mm_HandSolder, symbol Device:C
- added C14: 0.1uF, Capacitor_SMD:C_1812_4532Metric_Pad1.57x3.40mm_HandSolder, symbol Device:C
- added C15: 10nF, Capacitor_SMD:C_1812_4532Metric_Pad1.57x3.40mm_HandSolder, symbol Device:C
- added R20, R21, R22: 10K, Resistor_SMD:R_0805_2012Metric_Pad1.20x1.40mm_HandSolder, symbol Device:R
- added VR1: AP7366-33W5-7, AP7366-33W5-7:SOT95P285X140-5N, symbol AP7366-33W5-7:AP7366-33W5-7
- C10: value 7.14nF -> 0.1uF; footprint Capacitor_SMD:C_1206_3216Metric_Pad1.33x1.80mm_HandSolder -> Capacitor_SMD:C_0603_1608Metric_Pad1.08x0.95mm_HandSolder
- R51, R52: value 5K -> 5.1K
Connections:
- net +3V3: now also C13.2, C14.2, C15.2, R20.1, R21.1, R22.1, VR1.5 (OUT); no longer C10.1, R5.1
- net GND: now also C13.1, C14.1, C15.1, VR1.2 (GND); no longer U3.5 (VIO), U3.6 (VDD)
- net at C3.1, J1.A4 (VBUS), J1.A9 (VBUS)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: now also VR1.1 (IN), VR1.3 (EN)
- net INTN: now reaches U1.14 (MTDI/GPIO12/ADC2_CH5)
- net INTN: now also R5.1
- new net: C10.1, U3.5 (VIO), U3.6 (VDD)
- new net PMODE0: R20.2, U2.45 (PMODE0)
- new net PMODE1: R21.2, U2.44 (PMODE1)
- new net PMODE2: R22.2, U2.43 (PMODE2)
- no-connect marks 46 -> 44
Other:
- moved on the sheet: R19
